Commit message: 显示地图和小车

File: src/racecar_description/urdf/racecar.urdf (robot description, URDF)
Before this commit: robot racecar, 3 links, 2 joints
Links:
- removed link rear_wheel_left
- removed link rear_wheel_right
Joints:
- removed joint rear_wheel_left_joint
- removed joint rear_wheel_right_joint
