Commit message: 111111

File: src/racecar_description/urdf/racecar.urdf.xacro (robot description, xacro)
@@ -1,62 +1,410 @@
 <?xml version="1.0"?>
-<robot name="racecar" xmlns:xacro="http://www.ros.org/wiki/xacro">
-  <!-- 车体 -->
+<!--
+FSAC直线加速赛车模型（修正版）
+- 适配3米锥筒间距
+- 激光雷达距离惯导2.4m，高度0.8m（任务要求）
+- 双电机后驱
+- 随机偏航角：±3度
+-->
+<robot name="fsac_vehicle" xmlns:xacro="http://www.ros.org/wiki/xacro">
+  <!-- =====================================================
+       车辆参数（小型化适配）
+       ===================================================== -->
+  <xacro:property name="wheelbase" value="1.2" />        <!-- 轴距1.2m -->
+  <xacro:property name="track_width" value="0.8" />      <!-- 轮距0.8m -->
+  <xacro:property name="wheel_radius" value="0.25" />    <!-- 车轮半径 -->
+  <xacro:property name="wheel_width" value="0.2" />      <!-- 车轮宽度 -->
+  <!-- 车身尺寸（小型化） -->
+  <xacro:property name="body_length" value="2.2" />      <!-- 车身长度2.2m -->
+  <xacro:property name="body_width" value="1.0" />       <!-- 车身宽度1.0m -->
+  <xacro:property name="body_height" value="0.8" />      <!-- 车身高度0.8m -->
+  <!-- 激光雷达偏移（任务要求：距离惯导2.4m，高度0.2m） -->
+  <xacro:property name="lidar_distance" value="2.4" />   <!-- 距离惯导2.4m -->
+  <xacro:property name="lidar_height" value="0.2" />     <!-- 高度0.2m -->
+  <!-- 假设雷达在车辆前方 -->
+  <xacro:property name="lidar_x_offset" value="${lidar_distance}" />
+  <xacro:property name="lidar_y_offset" value="0" />
+  <xacro:property name="lidar_z_offset" value="${lidar_height}" />
+  <!-- =====================================================
+       材料定义
+       ===================================================== -->
+  <material name="red">
+    <color rgba="0.8 0.0 0.0 1.0"/>
+  </material>
+  <material name="blue">
+    <color rgba="0.0 0.0 0.8 1.0"/>
+  </material>
+  <material name="black">
+    <color rgba="0.1 0.1 0.1 1.0"/>
+  </material>
+  <material name="white">
+    <color rgba="0.9 0.9 0.9 1.0"/>
+  </material>
+  <material name="green">
+    <color rgba="0.0 0.8 0.0 1.0"/>
+  </material>
+  <!-- =====================================================
+       基础坐标系（惯导位置）
+       ===================================================== -->
   <link name="base_link">
     <visual>
-      <geometry>
-        <box size="0.5 0.3 0.1"/>
-      </geometry>
-      <material name="blue">
-        <color rgba="0.1 0.1 1.0 1.0"/>
-      </material>
-    </visual>
-    <collision>
-      <geometry>
-        <box size="0.5 0.3 0.1"/>
-      </geometry>
-    </collision>
-    <inertial>
-      <mass value="10"/>
-      <inertia ixx="0.1" ixy="0.0" ixz="0.0" iyy="0.1" iyz="0.0" izz="0.1"/>
-    </inertial>
-  </link>
-  <!-- Gazebo插件：只用虚拟轮子名驱动 -->
+      <origin xyz="0 0 0.4" rpy="0 0 0"/>
+      <geometry>
+        <box size="${body_length} ${body_width} ${body_height}"/>
+      </geometry>
+      <material name="red"/>
+    </visual>
+    <collision>
+      <origin xyz="0 0 0.4" rpy="0 0 0"/>
+      <geometry>
+        <box size="${body_length} ${body_width} ${body_height}"/>
+      </geometry>
+    </collision>
+    <inertial>
+      <origin xyz="0 0 0.4" rpy="0 0 0"/>
+      <mass value="300.0"/>
+      <inertia ixx="50" ixy="0" ixz="0" iyy="80" iyz="0" izz="100"/>
+    </inertial>
+  </link>
+  <!-- =====================================================
+       惯导传感器（IMU）- 标记惯导位置
+       ===================================================== -->
+  <joint name="imu_joint" type="fixed">
+    <parent link="base_link"/>
+    <child link="imu_link"/>
+    <origin xyz="0 0 0.2" rpy="0 0 0"/>  <!-- 惯导在base_link中心稍上方 -->
+  </joint>
+  <link name="imu_link">
+    <visual>
+      <origin xyz="0 0 0" rpy="0 0 0"/>
+      <geometry>
+        <box size="0.1 0.1 0.05"/>  <!-- 小盒子标记惯导位置 -->
+      </geometry>
+      <material name="green"/>
+    </visual>
+    <collision>
+      <origin xyz="0 0 0" rpy="0 0 0"/>
+      <geometry>
+        <box size="0.1 0.1 0.05"/>
+      </geometry>
+    </collision>
+    <inertial>
+      <origin xyz="0 0 0" rpy="0 0 0"/>
+      <mass value="0.5"/>
+      <inertia ixx="0.01" ixy="0" ixz="0" iyy="0.01" iyz="0" izz="0.01"/>
+    </inertial>
+  </link>
+  <!-- =====================================================
+       前轮（转向轮）
+       ===================================================== -->
+  <!-- 左前轮 -->
+  <joint name="front_left_wheel_joint" type="revolute">
+    <parent link="base_link"/>
+    <child link="front_left_wheel_link"/>
+    <origin xyz="${wheelbase/2} ${track_width/2} 0" rpy="0 0 0"/>
+    <axis xyz="0 0 1"/>
+    <limit lower="-0.6" upper="0.6" effort="50" velocity="10"/>
+  </joint>
+  <link name="front_left_wheel_link">
+    <visual>
+      <origin xyz="0 0 0" rpy="1.5708 0 0"/>
+      <geometry>
+        <cylinder radius="${wheel_radius}" length="${wheel_width}"/>
+      </geometry>
+      <material name="black"/>
+    </visual>
+    <collision>
+      <origin xyz="0 0 0" rpy="1.5708 0 0"/>
+      <geometry>
+        <cylinder radius="${wheel_radius}" length="${wheel_width}"/>
+      </geometry>
+    </collision>
+    <inertial>
+      <origin xyz="0 0 0" rpy="0 0 0"/>
+      <mass value="8.0"/>
+      <inertia ixx="0.5" ixy="0" ixz="0" iyy="0.5" iyz="0" izz="1"/>
+    </inertial>
+  </link>
+  <!-- 右前轮 -->
+  <joint name="front_right_wheel_joint" type="revolute">
+    <parent link="base_link"/>
+    <child link="front_right_wheel_link"/>
+    <origin xyz="${wheelbase/2} ${-track_width/2} 0" rpy="0 0 0"/>
+    <axis xyz="0 0 1"/>
+    <limit lower="-0.6" upper="0.6" effort="50" velocity="10"/>
+  </joint>
+  <link name="front_right_wheel_link">
+    <visual>
+      <origin xyz="0 0 0" rpy="1.5708 0 0"/>
+      <geometry>
+        <cylinder radius="${wheel_radius}" length="${wheel_width}"/>
+      </geometry>
+      <material name="black"/>
+    </visual>
+    <collision>
+      <origin xyz="0 0 0" rpy="1.5708 0 0"/>
+      <geometry>
+        <cylinder radius="${wheel_radius}" length="${wheel_width}"/>
+      </geometry>
+    </collision>
+    <inertial>
+      <origin xyz="0 0 0" rpy="0 0 0"/>
+      <mass value="8.0"/>
+      <inertia ixx="0.5" ixy="0" ixz="0" iyy="0.5" iyz="0" izz="1"/>
+    </inertial>
+  </link>
+  <!-- =====================================================
+       后轮（驱动轮 - 双电机后驱）
+       ===================================================== -->
+  <!-- 左后轮 -->
+  <joint name="rear_left_wheel_joint" type="continuous">
+    <parent link="base_link"/>
+    <child link="rear_left_wheel_link"/>
+    <origin xyz="${-wheelbase/2} ${track_width/2} 0" rpy="0 0 0"/>
+    <axis xyz="0 1 0"/>
+  </joint>
+  <link name="rear_left_wheel_link">
+    <visual>
+      <origin xyz="0 0 0" rpy="1.5708 0 0"/>
+      <geometry>
+        <cylinder radius="${wheel_radius}" length="${wheel_width}"/>
+      </geometry>
+      <material name="black"/>
+    </visual>
+    <collision>
+      <origin xyz="0 0 0" rpy="1.5708 0 0"/>
+      <geometry>
+        <cylinder radius="${wheel_radius}" length="${wheel_width}"/>
+      </geometry>
+    </collision>
+    <inertial>
+      <origin xyz="0 0 0" rpy="0 0 0"/>
+      <mass value="10.0"/>
+      <inertia ixx="0.8" ixy="0" ixz="0" iyy="0.8" iyz="0" izz="1.5"/>
+    </inertial>
+  </link>
+  <!-- 右后轮 -->
+  <joint name="rear_right_wheel_joint" type="continuous">
+    <parent link="base_link"/>
+    <child link="rear_right_wheel_link"/>
+    <origin xyz="${-wheelbase/2} ${-track_width/2} 0" rpy="0 0 0"/>
+    <axis xyz="0 1 0"/>
+  </joint>
+  <link name="rear_right_wheel_link">
+    <visual>
+      <origin xyz="0 0 0" rpy="1.5708 0 0"/>
+      <geometry>
+        <cylinder radius="${wheel_radius}" length="${wheel_width}"/>
+      </geometry>
+      <material name="black"/>
+    </visual>
+    <collision>
+      <origin xyz="0 0 0" rpy="1.5708 0 0"/>
+      <geometry>
+        <cylinder radius="${wheel_radius}" length="${wheel_width}"/>
+      </geometry>
+    </collision>
+    <inertial>
+      <origin xyz="0 0 0" rpy="0 0 0"/>
+      <mass value="10.0"/>
+      <inertia ixx="0.8" ixy="0" ixz="0" iyy="0.8" iyz="0" izz="1.5"/>
+    </inertial>
+  </link>
+  <!-- =====================================================
+       传感器：激光雷达（距离惯导2.4m，高度0.8m）
+       ===================================================== -->
+  <joint name="lidar_joint" type="fixed">
+    <parent link="base_link"/>
+    <child link="lidar_link"/>
+    <!-- 距离惯导2.4m，高度0.8m（任务要求） -->
+    <origin xyz="${lidar_x_offset} ${lidar_y_offset} ${lidar_z_offset}" rpy="0 0 0"/>
+  </joint>
+  <link name="lidar_link">
+    <visual>
+      <origin xyz="0 0 0" rpy="0 0 0"/>
+      <geometry>
+        <cylinder radius="0.08" length="0.15"/>
+      </geometry>
+      <material name="blue"/>
+    </visual>
+    <collision>
+      <origin xyz="0 0 0" rpy="0 0 0"/>
+      <geometry>
+        <cylinder radius="0.08" length="0.15"/>
+      </geometry>
+    </collision>
+    <inertial>
+      <origin xyz="0 0 0" rpy="0 0 0"/>
+      <mass value="1.5"/>
+      <inertia ixx="0.05" ixy="0" ixz="0" iyy="0.05" iyz="0" izz="0.05"/>
+    </inertial>
+  </link>
+  <!-- =====================================================
+       雷达支撑结构（可视化距离关系）
+       ===================================================== -->
+  <joint name="lidar_support_joint" type="fixed">
+    <parent link="base_link"/>
+    <child link="lidar_support_link"/>
+    <origin xyz="${lidar_distance/2} 0 ${lidar_height/2}" rpy="0 0 0"/>
+  </joint>
+  <link name="lidar_support_link">
+    <visual>
+      <origin xyz="0 0 0" rpy="0 0 0"/>
+      <geometry>
+        <box size="${lidar_distance} 0.03 0.03"/>  <!-- 细杆连接惯导和雷达 -->
+      </geometry>
+      <material name="white"/>
+    </visual>
+    <collision>
+      <origin xyz="0 0 0" rpy="0 0 0"/>
+      <geometry>
+        <box size="${lidar_distance} 0.03 0.03"/>
+      </geometry>
+    </collision>
+    <inertial>
+      <origin xyz="0 0 0" rpy="0 0 0"/>
+      <mass value="1.0"/>
+      <inertia ixx="0.1" ixy="0" ixz="0" iyy="0.2" iyz="0" izz="0.2"/>
+    </inertial>
+  </link>
+  <!-- =====================================================
+       距离标记（可视化2.4m距离）
+       ===================================================== -->
+  <joint name="distance_marker_joint" type="fixed">
+    <parent link="base_link"/>
+    <child link="distance_marker_link"/>
+    <origin xyz="${lidar_distance/2} 0 0.1" rpy="0 0 0"/>
+  </joint>
+  <link name="distance_marker_link">
+    <visual>
+      <origin xyz="0 0 0" rpy="0 0 0"/>
+      <geometry>
+        <box size="0.05 0.2 0.05"/>  <!-- 距离标记 -->
+      </geometry>
+      <material name="green"/>
+    </visual>
+    <inertial>
+      <origin xyz="0 0 0" rpy="0 0 0"/>
+      <mass value="0.1"/>
+      <inertia ixx="0.01" ixy="0" ixz="0" iyy="0.01" iyz="0" izz="0.01"/>
+    </inertial>
+  </link>
+  <!-- =====================================================
+       Gazebo插件：车辆控制
+       ===================================================== -->
   <gazebo>
-    <plugin name="differential_drive_controller" filename="libgazebo_ros_diff_drive.so">
-      <alwaysOn>true</alwaysOn>
-      <updateRate>100</updateRate>
-      <leftJoint>left_wheel_joint</leftJoint>
-      <rightJoint>right_wheel_joint</rightJoint>
-      <wheelSeparation>0.3</wheelSeparation>
-      <wheelDiameter>0.1</wheelDiameter>
-      <wheelTorque>20</wheelTorque>
-      <wheelAcceleration>1.0</wheelAcceleration>
-      <commandTopic>cmd_vel</commandTopic>
+    <plugin name="ackermann_drive_controller" filename="libgazebo_ros_ackermann_drive.so">
+      <commandTopic>ackermann_cmd</commandTopic>
       <odometryTopic>odom</odometryTopic>
       <odometryFrame>odom</odometryFrame>
+      <odometrySource>world</odometrySource>
+      <publishOdomTF>true</publishOdomTF>
       <robotBaseFrame>base_link</robotBaseFrame>
+      <publishWheelTF>false</publishWheelTF>
       <publishTf>true</publishTf>
-      <publishWheelTF>false</publishWheelTF>
-      <publishOdomTF>true</publishOdomTF>
       <publishWheelJointState>true</publishWheelJointState>
-      <legacyMode>false</legacyMode>
-      <odometrySource>world</odometrySource>
-      <rosDebugLevel>na</rosDebugLevel>
+      <frontLeftJoint>front_left_wheel_joint</frontLeftJoint>
+      <frontRightJoint>front_right_wheel_joint</frontRightJoint>
+      <rearLeftJoint>rear_left_wheel_joint</rearLeftJoint>
+      <rearRightJoint>rear_right_wheel_joint</rearRightJoint>
+      <wheelSeparation>${track_width}</wheelSeparation>
+      <wheelBase>${wheelbase}</wheelBase>
+      <wheelDiameter>${2*wheel_radius}</wheelDiameter>
+      <!-- 小型车性能参数 -->
+      <maxSteerAngle>0.6</maxSteerAngle>
+      <maxSpeed>12.0</maxSpeed>
+      <maxForce>2000.0</maxForce>
+      <!-- 物理参数 -->
+      <torque>800</torque>
+      <topicName>ackermann_cmd</topicName>
     </plugin>
   </gazebo>
-  <!-- 虚拟轮子关节（必须有，否则插件会报错） -->
-  <joint name="left_wheel_joint" type="continuous">
-    <parent link="base_link"/>
-    <child link="left_wheel"/>
-    <origin xyz="0 0.15 0" rpy="0 0 0"/>
-    <axis xyz="0 1 0"/>
-  </joint>
-  <joint name="right_wheel_joint" type="continuous">
-    <parent link="base_link"/>
-    <child link="right_wheel"/>
-    <origin xyz="0 -0.15 0" rpy="0 0 0"/>
-    <axis xyz="0 1 0"/>
-  </joint>
-  <link name="left_wheel"/>
-  <link name="right_wheel"/>
+  <!-- =====================================================
+       Gazebo插件：激光雷达
+       ===================================================== -->
+  <gazebo reference="lidar_link">
+    <material>Gazebo/Blue</material>
+    <sensor type="ray" name="lidar_sensor">
+      <pose>0 0 0 0 0 0</pose>
+      <visualize>true</visualize>
+      <update_rate>20</update_rate>
+      <ray>
+        <scan>
+          <horizontal>
+            <samples>360</samples>
+            <resolution>1</resolution>
+            <min_angle>-3.14159</min_angle>
+            <max_angle>3.14159</max_angle>
+          </horizontal>
+        </scan>
+        <range>
+          <min>0.2</min>
+          <max>30.0</max>
+          <resolution>0.01</resolution>
+        </range>
+        <noise>
+          <type>gaussian</type>
+          <mean>0.0</mean>
+          <stddev>0.01</stddev>
+        </noise>
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